File: audio.kicad_sch (KiCad schematic)
At the start: 34 parts, among them J3 USB_C_AUDIO, U10 TLV75533PDBVR, U11 PCM2903CDBR, Y2 12MHz

Commit message: Footprints: TVP7002 pad and vias per the OSSC, FX3 pads per AN70707; spare boot EEPROM
Parts:
- removed U10: TLV75533PDBVR, Package_TO_SOT_SMD:SOT-23-5, symbol Regulator_Linear:TLV75533PDBV
- removed U11: PCM2903CDBR, Package_SO:SSOP-28_5.3x10.2mm_P0.65mm, symbol ps1-av-capture:PCM2903C
- added U11: TLV75533PDBVR, Package_TO_SOT_SMD:SOT-23-5, symbol Regulator_Linear:TLV75533PDBV
- added U12: PCM2903CDBR, Package_SO:SSOP-28_5.3x10.2mm_P0.65mm, symbol ps1-av-capture:PCM2903C
Connections:
- net +3V3_AUD: now also U11.5 (OUT), U12.10 (VCCC), U12.17 (VCCP1), U12.19 (VCCP2), U12.23 (VCCX), U12.27 (VDD), U12.3 (VBUS), U12.8 (SEL0)
- net AUD_DM: now also U12.2 (D-)
- net AUD_DP: now also U12.1 (D+)
- net AUD_SEL1: now also U12.9 (SEL1)
- net AUD_VCOM: now also U12.14 (VCOM)
- net AUD_VINL: now also U12.12 (VINL)
- net AUD_VINR: now also U12.13 (VINR)
- net AUD_XI: now also U12.21 (XTI)
- net AUD_XO: now also U12.20 (XTO)
- net GND: now also U11.2 (GND), U12.11 (AGNDC), U12.18 (AGNDP), U12.22 (AGNDX), U12.26 (DGND), U12.4 (DGNDU)
- net VBUS_AUD: now also U11.1 (IN), U11.3 (EN)

Commit message: Status LED: common-anode RGB on FX3 GPIO50-52, firmware state map
XL-1615RGBC-RF (C965840) replaces the GPIO57 debug LED. Its LCSC pattern
numbers G and B the other way from the datasheet; fix_footprints.py renumbers
them and applies the datasheet's land pattern. GPIO budget in docs/design.md.
Parts:
- removed R63, R64: 5.1k, Resistor_SMD:R_0402_1005Metric, symbol Device:R
- added R73, R74: 10k, Resistor_SMD:R_0402_1005Metric, symbol Device:R
- R65, R66: value 22 -> 5.1k; LCSC C25092 -> C25905
- R67: value 1.5k -> 22; LCSC C25867 -> C25092
- R68: value 1M -> 22; LCSC C26083 -> C25092
- R69: value 1M -> 1.5k; LCSC C26083 -> C25867
- R71, R72: value 10k -> 1M; LCSC C25744 -> C26083
Connections:
- net +3V3_AUD: now also R69.2; no longer R67.2
- net AIN_L_C: now also R73.1; no longer R71.1
- net AIN_R_C: now also R74.1; no longer R72.1
- net AUD_CC1: now also R65.1
- net AUD_CC2: now also R66.1
- net AUD_DM: now also R68.2; no longer R66.2
- net AUD_DM_C: now also R68.1; no longer R66.1
- net AUD_DP: now also R67.2; no longer R65.2
- net AUD_DP_C: now also R69.1; no longer R65.1
- net AUD_SEL1: now also R70.2, R71.1; no longer R68.2, R69.1
- net AUD_VINL: now also R73.2; no longer R71.2
- net AUD_VINR: now also R74.2; no longer R72.2
- net AUD_XI: now also R72.1; no longer R70.1
- net AUD_XO: now also R72.2; no longer R70.2
- net GND: now also R65.2, R66.2, R71.2; no longer R69.2
- net VBUS_AUD: now also R70.1; no longer R68.1
